File: graphics/sources/eagle/60-hv-amp-digital-switching.sch (EAGLE design)
At the start: 12 parts, among them T1 BC547, X1 15V, X2 15V

Commit message: Fixed some Eagle graphics and added top and bottom board views to Chapter 6
Changed lines of the file:
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@@
 <setting verticaltext="up"/>
 </settings>
-<grid distance="0.1" unitdist="inch" unit="inch" style="lines" multiple="1" display="yes" altdistance="0.025" altunitdist="inch" altunit="inch"/>
+<grid distance="0.1" unitdist="inch" unit="inch" style="lines" multiple="1" display="no" altdistance="0.025" altunitdist="inch" altunit="inch"/>
 <layers>
 <layer number="91" name="Nets" color="34" fill="1" visible="yes" active="yes"/>
@@
 </plain>
 <instances>
-<instance part="N1" gate="A" x="43.18" y="35.56"/>
-<instance part="T1" gate="A" x="93.98" y="27.94"/>
+<instance part="N1" gate="A" x="43.18" y="35.56" smashed="yes">
+<attribute name="VALUE" x="40.64" y="39.37" size="1.524" layer="96" font="vector"/>
+</instance>
+<instance part="T1" gate="A" x="93.98" y="27.94" smashed="yes"/>
 <instance part="R1" gate="A" x="76.2" y="35.56"/>
 <instance part="R2" gate="A" x="91.44" y="20.32"/>
-<instance part="D1" gate="A" x="104.14" y="27.94" rot="R90"/>
-<instance part="N3" gate="A" x="60.96" y="38.1"/>
+<instance part="D1" gate="A" x="104.14" y="27.94" smashed="yes" rot="R90">
+<attribute name="VALUE" x="107.6325" y="26.035" size="1.524" layer="96" font="vector" rot="R90"/>
+</instance>
+<instance part="N3" gate="A" x="60.96" y="38.1" smashed="yes"/>
 <instance part="X1" gate="A" x="50.8" y="45.72"/>
-<instance part="D2" gate="A" x="142.24" y="27.94" rot="R90"/>
-<instance part="D3" gate="A" x="142.24" y="43.18" rot="R90"/>
+<instance part="D2" gate="A" x="142.24" y="27.94" smashed="yes" rot="R90">
+<attribute name="VALUE" x="145.7325" y="26.035" size="1.524" layer="96" font="vector" rot="R90"/>
+</instance>
+<instance part="D3" gate="A" x="142.24" y="43.18" smashed="yes" rot="R90">
+<attribute name="VALUE" x="145.7325" y="41.275" size="1.524" layer="96" font="vector" rot="R90"/>
+</instance>
 <instance part="$1" gate="A" x="142.24" y="15.24"/>
 <instance part="R3" gate="A" x="149.86" y="43.18" rot="R90"/>
 <instance part="X2" gate="A" x="142.24" y="55.88"/>
-<instance part="N2" gate="A" x="160.02" y="35.56" rot="MR90"/>
+<instance part="N2" gate="A" x="160.02" y="35.56" smashed="yes" rot="MR90"/>
 </instances>
 <busses>

Commit message: Added annotations to Eagle diagrams. Still needs textual updates.
Other:
- note added: "DIGITAL CONTROL INPUT"
- note added: "DIGITAL SWITCH"
- note added: "INVERTER"
- note added: "OPTOCOUPLER"
- note added: "PULL-UP RESISTOR"
- note added: "TRANSISTOR"
Changed lines of the file:
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@@
 <plain>
 <wire x1="121.92" y1="71.12" x2="121.92" y2="10.16" width="0.1524" layer="97" style="longdash"/>
-<text x="76.2" y="66.04" size="2.54" layer="97" font="vector" align="center">DIGITAL OUTPUT CARD</text>
-<text x="160.02" y="66.04" size="2.54" layer="97" font="vector" align="center">HV AMPLIFIER</text>
+<text x="66.04" y="66.04" size="3.81" layer="97" font="vector" align="center">DIGITAL OUTPUT CARD</text>
+<text x="172.72" y="66.04" size="3.81" layer="97" font="vector" align="center">HV AMPLIFIER</text>
+<text x="60.96" y="30.48" size="2.54" layer="97" font="vector" align="center">OPTOCOUPLER</text>
+<text x="35.56" y="43.18" size="2.54" layer="97" font="vector" align="center">INVERTER</text>
+<text x="96.52" y="15.24" size="2.54" layer="97" font="vector" align="center">TRANSISTOR</text>
+<text x="195.58" y="35.56" size="2.54" layer="97" font="vector" align="center">DIGITAL
+SWITCH</text>
+<text x="162.56" y="43.18" size="2.54" layer="97" font="vector" align="center">PULL-UP
+RESISTOR</text>
+<text x="17.78" y="25.4" size="2.54" layer="97" font="vector" align="center">DIGITAL
+CONTROL
+INPUT</text>
 </plain>
 <instances>
-<instance part="N1" gate="A" x="43.18" y="35.56" smashed="yes">
-<attribute name="VALUE" x="40.64" y="39.37" size="1.524" layer="96" font="vector"/>
+<instance part="N1" gate="A" x="35.56" y="35.56" smashed="yes">
+<attribute name="VALUE" x="33.02" y="39.37" size="1.524" layer="96" font="vector"/>
 </instance>
 <instance part="T1" gate="A" x="93.98" y="27.94" smashed="yes"/>
@@
 <instance part="R3" gate="A" x="149.86" y="43.18" rot="R90"/>
 <instance part="X2" gate="A" x="142.24" y="55.88"/>
-<instance part="N2" gate="A" x="160.02" y="35.56" smashed="yes" rot="MR90"/>
+<instance part="N2" gate="A" x="180.34" y="35.56" smashed="yes" rot="MR90"/>
 </instances>
 <busses>
@@
 <segment>
 <pinref part="N1" gate="A" pin="O"/>
-<wire x1="53.34" y1="35.56" x2="50.8" y2="35.56" width="0.1524" layer="91"/>
+<wire x1="53.34" y1="35.56" x2="43.18" y2="35.56" width="0.1524" layer="91"/>
 <pinref part="N3" gate="A" pin="C"/>
 </segment>
@@
 <segment>
 <pinref part="N1" gate="A" pin="I"/>
-<wire x1="38.1" y1="35.56" x2="35.56" y2="35.56" width="0.1524" layer="91"/>
-<label x="35.56" y="35.56" size="1.27" layer="95" font="vector" rot="R180" xref="yes"/>
+<wire x1="30.48" y1="35.56" x2="27.94" y2="35.56" width="0.1524" layer="91"/>
+<label x="27.94" y="35.56" size="1.27" layer="95" font="vector" rot="R180" xref="yes"/>
 </segment>
 </net>
@@
 <wire x1="149.86" y1="35.56" x2="149.86" y2="38.1" width="0.1524" layer="91"/>
 <pinref part="N2" gate="A" pin="D"/>
-<wire x1="149.86" y1="35.56" x2="154.94" y2="35.56" width="0.1524" layer="91"/>
+<wire x1="149.86" y1="35.56" x2="175.26" y2="35.56" width="0.1524" layer="91"/>
 <junction x="149.86" y="35.56"/>
 </segment>
@@
 <label x="137.16" y="50.8" size="1.27" layer="95" font="vector" rot="R180" xref="yes"/>
 <junction x="142.24" y="50.8"/>
-<pinref part="R3" gate="A" pin="N$DUMMY@2"/>
-<wire x1="149.86" y1="50.8" x2="149.86" y2="48.26" width="0.1524" layer="91"/>
-<junction x="149.86" y="50.8"/>
 <wire x1="149.86" y1="50.8" x2="142.24" y2="50.8" width="0.1524" layer="91"/>
 <pinref part="X2" gate="A" pin="1"/>
 <wire x1="142.24" y1="50.8" x2="142.24" y2="55.88" width="0.1524" layer="91"/>
+<pinref part="R3" gate="A" pin="N$DUMMY@2"/>
+<wire x1="149.86" y1="48.26" x2="149.86" y2="50.8" width="0.1524" layer="91"/>
 </segment>
 </net>
@@
 <segment>
 <pinref part="N2" gate="A" pin="S1"/>
-<wire x1="160.02" y1="27.94" x2="160.02" y2="20.32" width="0.1524" layer="91"/>
-<wire x1="160.02" y1="20.32" x2="175.26" y2="20.32" width="0.1524" layer="91"/>
-<label x="175.26" y="20.32" size="1.27" layer="95" font="vector" xref="yes"/>
+<wire x1="180.34" y1="27.94" x2="180.34" y2="20.32" width="0.1524" layer="91"/>
+<wire x1="180.34" y1="20.32" x2="195.58" y2="20.32" width="0.1524" layer="91"/>
+<label x="195.58" y="20.32" size="1.27" layer="95" font="vector" xref="yes"/>
 </segment>
 </net>
@@
 <segment>
 <pinref part="N2" gate="A" pin="S2B"/>
-<wire x1="160.02" y1="43.18" x2="160.02" y2="50.8" width="0.1524" layer="91"/>
-<wire x1="160.02" y1="50.8" x2="175.26" y2="50.8" width="0.1524" layer="91"/>
-<label x="175.26" y="50.8" size="1.27" layer="95" font="vector" xref="yes"/>
+<wire x1="180.34" y1="43.18" x2="180.34" y2="50.8" width="0.1524" layer="91"/>
+<wire x1="180.34" y1="50.8" x2="195.58" y2="50.8" width="0.1524" layer="91"/>
+<label x="195.58" y="50.8" size="1.27" layer="95" font="vector" xref="yes"/>
 </segment>
 </net>
@@
 <segment>
 <pinref part="N2" gate="A" pin="S2A"/>
-<wire x1="162.56" y1="43.18" x2="162.56" y2="48.26" width="0.1524" layer="91"/>
-<wire x1="162.56" y1="48.26" x2="175.26" y2="48.26" width="0.1524" layer="91"/>
-<label x="175.26" y="48.26" size="1.27" layer="95" font="vector" xref="yes"/>
+<wire x1="182.88" y1="43.18" x2="182.88" y2="48.26" width="0.1524" layer="91"/>
+<wire x1="182.88" y1="48.26" x2="195.58" y2="48.26" width="0.1524" layer="91"/>
+<label x="195.58" y="48.26" size="1.27" layer="95" font="vector" xref="yes"/>
 </segment>
 </net>
@@
 </schematic>
 </drawing>
+<compatibility>
+<note version="6.3" minversion="6.2.2" severity="warning">
+Since Version 6.2.2 text objects can contain more than one line,
+which will not be processed correctly with this version.
+</note>
+</compatibility>
 </eagle>

Commit message: Tweaks to digital switching figure
Connections:
- net UNWHITENED_INPUT renamed NORMAL_INPUT
- net WHITENED_INPUT renamed DEWHITENED_INPUT
Other:
- note added: "ANALOGUE INPUTS"
- note added: "ANALOGUE OUTPUT"
- note added: "SWITCH CONTROL INPUT"
Changed lines of the file:
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@@
 CONTROL
 INPUT</text>
+<text x="165.1" y="27.94" size="2.54" layer="97" font="vector" align="center">SWITCH
+CONTROL
+INPUT</text>
+<text x="203.2" y="58.42" size="2.54" layer="97" font="vector" align="center">ANALOGUE
+INPUTS</text>
+<text x="203.2" y="12.7" size="2.54" layer="97" font="vector" align="center">ANALOGUE
+OUTPUT</text>
 </plain>
 <instances>
@@
 </segment>
 </net>
-<net name="WHITENED_INPUT" class="0">
+<net name="DEWHITENED_INPUT" class="0">
 <segment>
 <pinref part="N2" gate="A" pin="S2B"/>
@@
 </segment>
 </net>
-<net name="UNWHITENED_INPUT" class="0">
+<net name="NORMAL_INPUT" class="0">
 <segment>
 <pinref part="N2" gate="A" pin="S2A"/>
